File: hardware/hundredsteppers.brd (EAGLE design)
At the start: 99.4 x 83.8 mm, 32 parts, among them IC1 74LS595N, IC2 74LS595N, IC3 74LS595N, IC4 74LS595N, IC5 74LS595N, IC6 74LS595N, X1 JST-XH-04-PIN-LONG-PAD, X10 JST-XH-04-PIN-LONG-PAD, X11 JST-XH-04-PIN-LONG-PAD, X12 JST-XH-04-PIN-LONG-PAD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

Commit message: only support 5-wires 4-phase stepper
Parts:
- removed X1, X10, X11, X12, X2, X3, X4, X5, X6, X7, X8, X9: JST-XH-04-PIN-LONG-PAD, JST_XH_Connectors:JST-XH-04-PACKAGE-LONG-PAD
- added U$1, U$10, U$11, U$12, U$2, U$3, U$4, U$5, U$6, U$7, U$8, U$9: JST-PH_5-PIN_HEADER, SRG:JST_B5B-PH_HEADER
- IC10, IC11, IC12, IC7, IC8, IC9: value (none) -> ULN2803A
- moved C3 3.59 mm to (85.1, 19.1)
- moved C5 3.59 mm to (34.3, 19.1)
- moved C6 3.59 mm to (59.7, 19.1)
- moved C1 2.54 mm to (35.6, 72.4)
- moved C2 2.54 mm to (61.0, 72.4)
- moved C4 2.54 mm to (10.2, 72.4)
- moved IC4 2.54 mm to (72.4, 17.8)
- moved IC11 2.54 mm to (48.3, 30.5)
- moved IC12 2.54 mm to (22.9, 30.5)
- moved IC5 2.54 mm to (47.0, 17.8)
- moved IC6 2.54 mm to (21.6, 17.8)
- moved IC10 2.54 mm to (73.7, 30.5)
Connections:
- net 0A: now also U$1.P1; no longer X1.1
- net 0B: now also U$1.P2; no longer X1.2
- net 0C: now also U$1.P3; no longer X1.3
- net 0D: now also U$1.P4; no longer X1.4
- net 10A: now also U$11.P1; no longer X11.1
- net 10B: now also U$11.P2; no longer X11.2
- net 10C: now also U$11.P3; no longer X11.3
- net 10D: now also U$11.P4; no longer X11.4
- net 11A: now also U$12.P1; no longer X12.1
- net 11B: now also U$12.P2; no longer X12.2
- net 11C: now also U$12.P3; no longer X12.3
- net 11D: now also U$12.P4; no longer X12.4
- net 1A: now also U$2.P1; no longer X2.1
- net 1B: now also U$2.P2; no longer X2.2
- net 1C: now also U$2.P3; no longer X2.3
- net 1D: now also U$2.P4; no longer X2.4
- net 2A: now also U$3.P1; no longer X3.1
- net 2B: now also U$3.P2; no longer X3.2
- net 2C: now also U$3.P3; no longer X3.3
- net 2D: now also U$3.P4; no longer X3.4
- net 3A: now also U$4.P1; no longer X4.1
- net 3B: now also U$4.P2; no longer X4.2
- net 3C: now also U$4.P3; no longer X4.3
- net 3D: now also U$4.P4; no longer X4.4
- net 4A: now also U$5.P1; no longer X5.1
- net 4B: now also U$5.P2; no longer X5.2
- net 4C: now also U$5.P3; no longer X5.3
- net 4D: now also U$5.P4; no longer X5.4
- net 5A: now also U$6.P1; no longer X6.1
- net 5B: now also U$6.P2; no longer X6.2
- net 5C: now also U$6.P3; no longer X6.3
- net 5D: now also U$6.P4; no longer X6.4
- net 6A: now also U$7.P1; no longer X7.1
- net 6B: now also U$7.P2; no longer X7.2
- net 6C: now also U$7.P3; no longer X7.3
- net 6D: now also U$7.P4; no longer X7.4
- net 7A: now also U$8.P1; no longer X8.1
- net 7B: now also U$8.P2; no longer X8.2
- net 7C: now also U$8.P3; no longer X8.3
- net 7D: now also U$8.P4; no longer X8.4
- net 8A: now also U$9.P1; no longer X9.1
- net 8B: now also U$9.P2; no longer X9.2
- net 8C: now also U$9.P3; no longer X9.3
- net 8D: now also U$9.P4; no longer X9.4
- net 9A: now also U$10.P1; no longer X10.1
- net 9B: now also U$10.P2; no longer X10.2
- net 9C: now also U$10.P3; no longer X10.3
- net 9D: now also U$10.P4; no longer X10.4
- net VCC: now also U$1.P5, U$10.P5, U$11.P5, U$12.P5, U$2.P5, U$3.P5, U$4.P5, U$5.P5, U$6.P5, U$7.P5, U$8.P5, U$9.P5
Routing:
- net VCC: track 473.3 -> 594.9 mm
- net SHCP: track 241.4 -> 233.8 mm
- net STCP: track 252.8 -> 245.2 mm
- net OUT3: track 98.7 -> 91.0 mm
- net 6A: track 11.7 -> 7.95 mm
- net 0A: track 11.7 -> 7.95 mm
- net 0B: track 11.7 -> 8.11 mm
- net 6B: track 11.7 -> 8.11 mm
- net 6C: track 11.0 -> 8.30 mm
- net 0C: track 11.0 -> 8.30 mm
- net DOUT: track 160.6 -> 158.0 mm
- net 0D: track 10.3 -> 8.52 mm
- net 6D: track 10.3 -> 8.52 mm
- net 2A: track 9.20 -> 7.95 mm
- net 8A: track 9.20 -> 7.95 mm
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Other:
- board text added: "Hundred Steppers v0.3 by Hank"
- board text removed: "Hundred Steppers v0.2 by Hank"
