File: hardware/hundredsteppers.sch (EAGLE design)
At the start: 32 parts, among them IC1 74LS595N, IC2 74LS595N, IC3 74LS595N, IC4 74LS595N, IC5 74LS595N, IC6 74LS595N, X1 JST-XH-04-PIN-LONG-PAD, X10 JST-XH-04-PIN-LONG-PAD, X11 JST-XH-04-PIN-LONG-PAD, X12 JST-XH-04-PIN-LONG-PAD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

Commit message: only support 5-wires 4-phase stepper
Parts:
- removed X1, X10, X11, X12, X2, X3, X4, X5, X6, X7, X8, X9: JST-XH-04-PIN-LONG-PAD, JST_XH_Connectors:JST-XH-04-PIN-LONG-PAD
- added U$1, U$10, U$11, U$12, U$2, U$3, U$4, U$5, U$6, U$7, U$8, U$9: JST-PH_5-PIN_HEADER, SRG:JST-PH_5-PIN_HEADER
- IC10, IC11, IC12, IC7, IC8, IC9: value (none) -> ULN2803A
Connections:
- net 0A: now also U$1.1; no longer X1-1.S
- net 0B: now also U$1.2; no longer X1-2.S
- net 0C: now also U$1.3; no longer X1-3.S
- net 0D: now also U$1.4; no longer X1-4.S
- net 10A: now also U$11.1; no longer X11-1.S
- net 10B: now also U$11.2; no longer X11-2.S
- net 10C: now also U$11.3; no longer X11-3.S
- net 10D: now also U$11.4; no longer X11-4.S
- net 11A: now also U$12.1; no longer X12-1.S
- net 11B: now also U$12.2; no longer X12-2.S
- net 11C: now also U$12.3; no longer X12-3.S
- net 11D: now also U$12.4; no longer X12-4.S
- net 1A: now also U$2.1; no longer X2-1.S
- net 1B: now also U$2.2; no longer X2-2.S
- net 1C: now also U$2.3; no longer X2-3.S
- net 1D: now also U$2.4; no longer X2-4.S
- net 2A: now also U$3.1; no longer X3-1.S
- net 2B: now also U$3.2; no longer X3-2.S
- net 2C: now also U$3.3; no longer X3-3.S
- net 2D: now also U$3.4; no longer X3-4.S
- net 3A: now also U$4.1; no longer X4-1.S
- net 3B: now also U$4.2; no longer X4-2.S
- net 3C: now also U$4.3; no longer X4-3.S
- net 3D: now also U$4.4; no longer X4-4.S
- net 4A: now also U$5.1; no longer X5-1.S
- net 4B: now also U$5.2; no longer X5-2.S
- net 4C: now also U$5.3; no longer X5-3.S
- net 4D: now also U$5.4; no longer X5-4.S
- net 5A: now also U$6.1; no longer X6-1.S
- net 5B: now also U$6.2; no longer X6-2.S
- net 5C: now also U$6.3; no longer X6-3.S
- net 5D: now also U$6.4; no longer X6-4.S
- net 6A: now also U$7.1; no longer X7-1.S
- net 6B: now also U$7.2; no longer X7-2.S
- net 6C: now also U$7.3; no longer X7-3.S
- net 6D: now also U$7.4; no longer X7-4.S
- net 7A: now also U$8.1; no longer X8-1.S
- net 7B: now also U$8.2; no longer X8-2.S
- net 7C: now also U$8.3; no longer X8-3.S
- net 7D: now also U$8.4; no longer X8-4.S
- net 8A: now also U$9.1; no longer X9-1.S
- net 8B: now also U$9.2; no longer X9-2.S
- net 8C: now also U$9.3; no longer X9-3.S
- net 8D: now also U$9.4; no longer X9-4.S
- net 9A: now also U$10.1; no longer X10-1.S
- net 9B: now also U$10.2; no longer X10-2.S
- net 9C: now also U$10.3; no longer X10-3.S
- net 9D: now also U$10.4; no longer X10-4.S
- net VCC: now also U$1.5, U$10.5, U$11.5, U$12.5, U$2.5, U$3.5, U$4.5, U$5.5, U$6.5, U$7.5, U$8.5, U$9.5
Other:
- moved on the sheet: INPUT, OUTPUT
